File: AD8232_Board.kicad_pcb (KiCad board)
At the start: 4 copper layers, 25.4 x 17.7 mm, 26 parts, among them J1 Conn_01x05_Pin, J2 Conn_01x05_Pin, U1 AD8232

Commit message: Update silkscreen and soldermask settings
Add multiple bottom silkscreen text labels (RL, AN, NC, LA, RA, 3.3, GND, SDN, LO+, LO-) to AD8232_Board.kicad_pcb and remove an explicit solder_mask_min_width entry. Adjust solder mask to copper clearance in AD8232_Board.kicad_pro from 0.0 to 0.005. Regenerate/update Gerber outputs (timestamps updated) and add the new bottom silkscreen Gerber (gerber/AD8232_Board-B_Silkscreen.gbo); updates to B_Mask and B_Paste files included as part of the export.
Other:
- board text added: "3.3"
- board text added: "AN"
- board text added: "GND"
- board text added: "LA"
- board text added: "LO+"
- board text added: "LO-"
- board text added: "NC"
- board text added: "RA"
- board text added: "RL"
- board text added: "SDN"
Changed lines of the file:
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@@
 		)
 		(pad_to_mask_clearance 0)
-		(solder_mask_min_width 0.12)
 		(allow_soldermask_bridges_in_footprints no)
 		(tenting
@@
 		(layer "Edge.Cuts")
 	)
+	(gr_text "RL"
+		(at 159.3 107.1 0)
+		(layer "B.SilkS")
+		(effects
+			(font
+				(size 0.5 0.5)
+				(thickness 0.125)
+				(bold yes)
+			)
+			(justify left bottom mirror)
+		)
+	)
+	(gr_text "AN"
+		(at 159.3 109.6 0)
+		(layer "B.SilkS")
+		(effects
+			(font
+				(size 0.5 0.5)
+				(thickness 0.125)
+				(bold yes)
+			)
+			(justify left bottom mirror)
+		)
+	)
+	(gr_text "NC"
+		(at 159.3 111.6 0)
+		(layer "B.SilkS")
+		(effects
+			(font
+				(size 0.5 0.5)
+				(thickness 0.125)
+				(bold yes)
+			)
+			(justify left bottom mirror)
+		)
+	)
+	(gr_text "LA"
+		(at 159.4 102 0)
+		(layer "B.SilkS")
+		(effects
+			(font
+				(size 0.5 0.5)
+				(thickness 0.125)
+				(bold yes)
+			)
+			(justify left bottom mirror)
+		)
+	)
+	(gr_text "RA"
+		(at 159.5 104.5 0)
+		(layer "B.SilkS")
+		(effects
+			(font
+				(size 0.5 0.5)
+				(thickness 0.125)
+				(bold yes)
+			)
+			(justify left bottom mirror)
+		)
+	)
+	(gr_text "3.3"
+		(at 177.7 102.6 0)
+		(layer "B.SilkS")
+		(effects
+			(font
+				(size 0.5 0.5)
+				(thickness 0.125)
+				(bold yes)
+			)
+			(justify left bottom mirror)
+		)
+	)
+	(gr_text "GND"
+		(at 177.7 105 0)
+		(layer "B.SilkS")
+		(effects
+			(font
+				(size 0.5 0.5)
+				(thickness 0.125)
+				(bold yes)
+			)
+			(justify left bottom mirror)
+		)
+	)
+	(gr_text "SDN"
+		(at 177.8 107.6 0)
+		(layer "B.SilkS")
+		(effects
+			(font
+				(size 0.5 0.5)
+				(thickness 0.125)
+				(bold yes)
+			)
+			(justify left bottom mirror)
+		)
+	)
+	(gr_text "LO+"
+		(at 177.8 110.1 0)
+		(layer "B.SilkS")
+		(effects
+			(font
+				(size 0.5 0.5)
+				(thickness 0.125)
+				(bold yes)
+			)
+			(justify left bottom mirror)
+		)
+	)
+	(gr_text "LO-\n"
+		(at 177.8 111.3 0)
+		(layer "B.SilkS")
+		(effects
+			(font
+				(size 0.5 0.5)
+				(thickness 0.125)
+				(bold yes)
+			)
+			(justify left bottom mirror)
+		)
+	)
 	(gr_text "AD8232\nECG MONITOR\nby\nEkenedirichukwu"
